File: ESP32-C6-RC.kicad_pcb (KiCad board)
At the start: 2 copper layers, 1 part

Commit message: update schemtics and pcb
Parts:
- added +V1: +V, TestPoint:TestPoint_THTPad_D1.5mm_Drill0.7mm, F.Cu at (93.8, 42.5)
- added A1: A, TestPoint:TestPoint_THTPad_D1.5mm_Drill0.7mm, F.Cu at (87.1, 42.6)
- added B1: B, TestPoint:TestPoint_THTPad_D1.5mm_Drill0.7mm, F.Cu at (83.8, 42.6)
- added C1: 100nF, Capacitor_SMD:C_0805_2012Metric_Pad1.18x1.45mm_HandSolder, F.Cu at (93.0, 48.4)
- added C2: 100nF, Capacitor_SMD:C_0805_2012Metric_Pad1.18x1.45mm_HandSolder, F.Cu at (93.0, 66.4)
- added C3: 100nF, Capacitor_SMD:C_0805_2012Metric_Pad1.18x1.45mm_HandSolder, F.Cu at (80.7, 58.5)
- added C4: 100nF, Capacitor_SMD:C_0805_2012Metric_Pad1.18x1.45mm_HandSolder, F.Cu at (82.7, 46.6)
- added C5: 22uF 10v, Capacitor_Tantalum_SMD:CP_EIA-3528-12_Kemet-T_HandSolder, F.Cu at (93.1, 55.1)
- added C6: 22uF 10v, Capacitor_Tantalum_SMD:CP_EIA-3528-12_Kemet-T_HandSolder, F.Cu at (88.6, 50.3)
- added D1: SS34, Diode_SMD:D_SMA, F.Cu at (87.9, 62.3)
- added FB1: MPZ2012S101AT000, Diode_SMD:D_0805_2012Metric_Pad1.15x1.40mm_HandSolder, F.Cu at (89.3, 46.3)
- added G1: G1, TestPoint:TestPoint_THTPad_D1.5mm_Drill0.7mm, F.Cu at (90.2, 42.5)
- added J3: Conn_01x03, Connector_PinHeader_2.54mm:PinHeader_1x03_P2.54mm_Vertical, F.Cu at (75.4, 42.5)
- added R1: 1k, Resistor_SMD:R_0805_2012Metric_Pad1.20x1.40mm_HandSolder, F.Cu at (86.1, 65.3)
- added R2: 10k, Resistor_SMD:R_0805_2012Metric_Pad1.20x1.40mm_HandSolder, F.Cu at (77.4, 47.4)
- added R3: 10k, Resistor_SMD:R_0805_2012Metric_Pad1.20x1.40mm_HandSolder, F.Cu at (77.0, 52.4)
- added R4: 330, Resistor_SMD:R_0805_2012Metric_Pad1.20x1.40mm_HandSolder, F.Cu at (74.6, 47.5)
- added R5: 330, Resistor_SMD:R_0805_2012Metric_Pad1.20x1.40mm_HandSolder, F.Cu at (75.5, 56.9)
- added SW1: SW_Push, myCustomLib:SW_SPST_B3S-1000, F.Cu at (78.6, 63.4)
- added U2: RZ7899, Package_SO:SOP-8_3.76x4.96mm_P1.27mm, F.Cu at (81.7, 52.3)
- added U3: AMS1117-5.0, Package_TO_SOT_SMD:SOT-89-3_Handsoldering, F.Cu at (88.1, 56.8)
- U1: value ~ -> ESP32-C6 zero; moved to B.Cu
- moved U1 49.2 mm to (85.0, 59.0), turned to 180 degrees
Connections:
- U1 pad 1: unconnected-(U1-VCC-Pad1) -> +5V
- U1 pad 14: unconnected-(U1-IO18-Pad14) -> PWM_OUT2
- U1 pad 15: unconnected-(U1-IO15-Pad15) -> PWM_OUT1
- U1 pad 16: unconnected-(U1-IO14-Pad16) -> SERVO_X
- U1 pad 2: unconnected-(U1-GND-Pad2) -> GND
- U1 pad 3: unconnected-(U1-V3V-Pad3) -> +3.3V
- U1 pad 8: unconnected-(U1-IO4-Pad8) -> Net-(U1-IO4)
Routing:
- net +3.3V: track 0.00 -> 35.8 mm, vias 0 -> 2
- net Net-(U3-VO): track 0.00 -> 28.1 mm
- net +7.4V: track 0.00 -> 26.9 mm, vias 0 -> 2
- net Net-(D1-A): track 0.00 -> 24.5 mm
- net +5V: track 0.00 -> 21.2 mm, vias 0 -> 1
- net Net-(U1-IO4): track 0.00 -> 20.1 mm, vias 0 -> 1
- net SERVO_X: track 0.00 -> 16.7 mm
- net Net-(U2-inr): track 0.00 -> 13.5 mm
- net Net-(U2-inf): track 0.00 -> 11.6 mm
- net PWM_OUT1: track 0.00 -> 10.9 mm, vias 0 -> 1
- net MOT-B: track 0.00 -> 10.6 mm
- net MOT-A: track 0.00 -> 10.4 mm
- net GND: track 0.00 -> 5.20 mm, vias 0 -> 1
- net PWM_OUT2: track 0.00 -> 5.09 mm, vias 0 -> 1
- added copper zone on B.Cu, net GND
- added copper zone on F.Cu, net GND
Other:
- board outline added: 23 x 32.5 mm

Commit message: fix pcb
Parts:
- moved G1 0.28 mm to (90.5, 42.5)
- moved A1 0.10 mm to (87.0, 42.6)
Routing:
- net SERVO_X: track 16.7 -> 15.2 mm
Changed lines of the file:
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@@
 		(tags "test point THT pad")
 		(property "Reference" "B1"
-			(at -0.5 1.775 0)
+			(at -0.08 1.775 0)
 			(layer "F.SilkS")
 			(effects
@@
 	(footprint "TestPoint:TestPoint_THTPad_D1.5mm_Drill0.7mm"
 		(layer "F.Cu")
-		(at 87.1 42.6 180)
+		(at 87 42.6 180)
 		(descr "THT pad as test Point, diameter 1.5mm, hole diameter 0.7mm")
 		(tags "test point THT pad")
 		(property "Reference" "A1"
-			(at -0.475 1.775 0)
+			(at -0.13 1.775 0)
 			(layer "F.SilkS")
 			(effects
@@
 	(footprint "TestPoint:TestPoint_THTPad_D1.5mm_Drill0.7mm"
 		(layer "F.Cu")
-		(at 90.2 42.5)
+		(at 90.48 42.49)
 		(descr "THT pad as test Point, diameter 1.5mm, hole diameter 0.7mm")
 		(tags "test point THT pad")
@@
 	)
 	(segment
-		(start 79.795 47.6)
-		(end 79.795 47.405)
+		(start 83.75 42.6)
+		(end 83.75 43.75)
 		(width 0.5)
 		(layer "F.Cu")
@@
 	)
 	(segment
-		(start 83.75 43.75)
-		(end 83.75 42.6)
+		(start 79.795 47.6)
+		(end 79.795 47.405)
 		(width 0.5)
 		(layer "F.Cu")
@@
 	)
 	(segment
-		(start 87.1 44)
-		(end 87.1 42.6)
+		(start 87 44.1)
+		(end 86.865 44.235)
+		(width 0.5)
+		(layer "F.Cu")
+		(net 5)
+	)
+	(segment
+		(start 87 42.6)
+		(end 87 44.1)
 		(width 0.5)
 		(layer "F.Cu")
@@
 	(segment
 		(start 84.5 46.6)
-		(end 87.1 44)
+		(end 86.865 44.235)
 		(width 0.5)
 		(layer "F.Cu")
@@
 	)
 	(segment
-		(start 75.4 44.075)
-		(end 75.4 42.5)
-		(width 0.2)
-		(layer "B.Cu")
-		(net 8)
-	)
-	(segment
 		(start 74.013 53.848)
 		(end 74.325 54.16)
@@
 	)
 	(segment
-		(start 79.565 54.16)
-		(end 79.6 54.16)
-		(width 0.2)
-		(layer "B.Cu")
-		(net 9)
-	)
-	(segment
 		(start 88.7 54.185)
 		(end 88.725 54.16)
@@
 	)
 	(segment
-		(start 73.775 58.325)
-		(end 74.2 57.9)
+		(start 73.84 59.25)
+		(end 73.84 58.26)
 		(width 0.5)
 		(layer "F.Cu")
@@
 	)
 	(segment
-		(start 73.775 59.25)
-		(end 73.775 58.325)
+		(start 75.1 57.9)
+		(end 75.2 57.8)
 		(width 0.5)
 		(layer "F.Cu")
@@
 	)
 	(segment
-		(start 75.1 57.9)
-		(end 75.2 57.8)
+		(start 74.2 57.9)
+		(end 75.1 57.9)
 		(width 0.5)
 		(layer "F.Cu")
@@
 	)
 	(segment
-		(start 74.2 57.9)
-		(end 75.1 57.9)
+		(start 73.84 58.26)
+		(end 74.2 57.9)
 		(width 0.5)
 		(layer "F.Cu")
@@
 	)
 	(via
-		(at 73.775 59.25)
+		(at 73.84 59.25)
 		(size 0.6)
 		(drill 0.3)
