File: ESP32-C6-RC.kicad_sch (KiCad schematic)
At the start: 19 parts, among them J1 Conn_01x02, J2 Conn_01x02, J3 Conn_01x03, SW1 SW_Push, U2 RZ7899, U3 AMS1117-5.0

Commit message: update schemtics and pcb
Parts:
- removed J1, J2: Conn_01x02, Connector_PinHeader_2.54mm:PinHeader_1x02_P2.54mm_Vertical, symbol Connector_Generic:Conn_01x02
- added +V1: +V, TestPoint:TestPoint_THTPad_D1.5mm_Drill0.7mm, symbol Connector:TestPoint_Small
- added A1: A, TestPoint:TestPoint_THTPad_D1.5mm_Drill0.7mm, symbol Connector:TestPoint_Small
- added B1: B, TestPoint:TestPoint_THTPad_D1.5mm_Drill0.7mm, symbol Connector:TestPoint_Small
- added FB1: MPZ2012S101AT000, Diode_SMD:D_0805_2012Metric_Pad1.15x1.40mm_HandSolder, symbol Device:FerriteBead_Small
- added G1: G1, TestPoint:TestPoint_THTPad_D1.5mm_Drill0.7mm, symbol Connector:TestPoint_Small
- D1: value US1M -> SS34
- SW1: footprint Button_Switch_SMD:SW_SPST_B3S-1000 -> myCustomLib:SW_SPST_B3S-1000
- U1: value ~ -> ESP32-C6 zero
- U2: footprint Package_SO:SOIC-8_5.3x5.3mm_P1.27mm -> Package_SO:SOP-8_3.76x4.96mm_P1.27mm
- U3: footprint Package_TO_SOT_SMD:SOT-223-3_TabPin2 -> Package_TO_SOT_SMD:SOT-89-3_Handsoldering
Connections:
- net +7.4V: now reaches C5.1
- net +7.4V: now also C1.1, C3.1, D1.1 (K), U2.4 (vcc), U3.3 (VI)
- net GND: now reaches C5.2
- net GND: now also C1.2, C2.2, C3.2, C6.2, J3.3 (Pin_3), SW1.1, U1.2 (GND), U2.3 (gnd), U3.1 (GND), G1.1
- net at C6.1: now also C2.1, U3.2 (VO), FB1.1
- net SERVO_X: now reaches J3.1 (Pin_1)
- net SERVO_X: now also U1.16 (IO14)
- net +5V: now reaches J3.2 (Pin_2)
- net +5V: now also U1.1 (VCC), FB1.2
- net PWM_OUT1: now reaches R4.1
- net PWM_OUT1: now also U1.15 (IO15)
- net at R4.2: now also R2.2, U2.1 (inr)
- net at SW1.2: now also R1.2, U1.8 (IO4)
- net PWM_OUT2: now reaches U1.14 (IO18)
- net PWM_OUT2: now also R5.1
- net +3.3V: now reaches U1.3 (V3V)
- net +3.3V: now also R1.1, R2.1, R3.2
- net MOT-A: now reaches C4.1
- net MOT-A: now also U2.5 (ouf), U2.6 (outf), A1.1
- net MOT-B: now reaches C4.2
- net MOT-B: now also U2.7 (outr), U2.8 (outr), B1.1
- net at R5.2: now also R3.1, U2.2 (inf)
- net at D1.2 (A): now also +V1.1
- no-connect marks 0 -> 11
Other:
- moved on the sheet: C1, C2, C3, C4, C5, C6, D1, R1, R2, R3, R4, R5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

Commit message: fix pcb
Changed lines of the file:
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@@
 		)
 	)
-	(wire
-		(pts
-			(xy 43.18 25.4) (xy 43.18 29.21)
-		)
-		(stroke
-			(width 0)
-			(type default)
-		)
-	)
 	(global_label "MOT-A"
 		(shape input)
@@
 	(symbol
 		(lib_id "power:PWR_FLAG")
-		(at 43.18 29.21 180)
-		(unit 1)
-		(exclude_from_sim no)
-		(in_bom yes)
-		(on_board yes)
-		(dnp no)
-		(fields_autoplaced yes)
-		(property "Reference" "#FLG03"
-			(at 43.18 31.115 0)
-			(effects
-				(font
-					(size 1.27 1.27)
-				)
-				(hide yes)
-			)
-		)
-		(property "Value" "PWR_FLAG"
-			(at 43.18 34.29 0)
-			(effects
-				(font
-					(size 1.27 1.27)
-				)
-			)
-		)
-		(property "Footprint" ""
-			(at 43.18 29.21 0)
-			(effects
-				(font
-					(size 1.27 1.27)
-				)
-				(hide yes)
-			)
-		)
-		(property "Datasheet" "~"
-			(at 43.18 29.21 0)
-			(effects
-				(font
-					(size 1.27 1.27)
-				)
-				(hide yes)
-			)
-		)
-		(property "Description" "Special symbol for telling ERC where power comes from"
-			(at 43.18 29.21 0)
-			(effects
-				(font
-					(size 1.27 1.27)
-				)
-				(hide yes)
-			)
-		)
-		(pin "1"
-		)
-		(instances
-			(project ""
-				(path "/c7efdda5-2cce-48fd-8ac9-1be4f59a0af3"
-					(reference "#FLG03")
-					(unit 1)
-				)
-			)
-		)
-	)
-	(symbol
-		(lib_id "power:PWR_FLAG")
 		(at 27.94 25.4 0)
 		(unit 1)
@@
 					(unit 1)
 				)
-			)
-		)
-	)
-	(symbol
-		(lib_id "power:+3V3")
-		(at 43.18 25.4 0)
-		(unit 1)
-		(exclude_from_sim no)
-		(in_bom yes)
-		(on_board yes)
-		(dnp no)
-		(fields_autoplaced yes)
-		(property "Reference" "#PWR023"
-			(at 43.18 29.21 0)
-			(effects
-				(font
-					(size 1.27 1.27)
-				)
-				(hide yes)
-			)
-		)
-		(property "Value" "+3V3"
-			(at 43.18 20.32 0)
-			(effects
-				(font
-					(size 1.27 1.27)
-				)
-			)
-		)
-		(property "Footprint" ""
-			(at 43.18 25.4 0)
-			(effects
-				(font
-					(size 1.27 1.27)
-				)
-				(hide yes)
-			)
-		)
-		(property "Datasheet" ""
-			(at 43.18 25.4 0)
-			(effects
-				(font
-					(size 1.27 1.27)
-				)
-				(hide yes)
-			)
-		)
-		(property "Description" "Power symbol creates a global label with name \"+3V3\""
-			(at 43.18 25.4 0)
-			(effects
-				(font
-					(size 1.27 1.27)
-				)
-				(hide yes)
-			)
-		)
-		(pin "1"
-		)
-		(instances
-			(project ""
-				(path "/c7efdda5-2cce-48fd-8ac9-1be4f59a0af3"
-					(reference "#PWR023")
-					(unit 1)
-				)
